File: zynqPCB/LCD50.kicad_sch (KiCad schematic)
At the start: 29 parts, among them J9 HDMI_A, Q10 IRLML2502, Q8 IRLML2502, Q9 IRLML2502, U20B xc7z020clg484, U20D xc7z020clg484, U20E xc7z020clg484, U21 PCA9306

Commit message: Update audio schematic
Parts:
- renumbered U20B to U20B1, U20D to U20D1, U20E to U20E1
Changed lines of the file:
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@@
 		(on_board yes)
 		(dnp no)
-		(property "Reference" "U20B"
+		(property "Reference" "U20B1"
 			(at 168.91 36.83 0)
 			(effects
@@
 			(project "DFTBoard"
 				(path "/49eba173-d38c-4d05-b21c-b4a14c4948c2/00000000-0000-0000-0000-00005c7c62ae"
-					(reference "U20B")
+					(reference "U20B1")
 					(unit 2)
 				)
@@
 		(on_board yes)
 		(dnp no)
-		(property "Reference" "U20D"
+		(property "Reference" "U20D1"
 			(at 223.52 36.83 0)
 			(effects
@@
 			(project "DFTBoard"
 				(path "/49eba173-d38c-4d05-b21c-b4a14c4948c2/00000000-0000-0000-0000-00005c7c62ae"
-					(reference "U20D")
+					(reference "U20D1")
 					(unit 4)
 				)
@@
 		(on_board yes)
 		(dnp no)
-		(property "Reference" "U20E"
+		(property "Reference" "U20E1"
 			(at 267.97 36.83 0)
 			(effects
@@
 			(project "DFTBoard"
 				(path "/49eba173-d38c-4d05-b21c-b4a14c4948c2/00000000-0000-0000-0000-00005c7c62ae"
-					(reference "U20E")
+					(reference "U20E1")
 					(unit 5)
 				)
