File: zynqPCB/USB.kicad_sch (KiCad schematic)
At the start: 47 parts, among them J6 USB_A, J7 USB_B, U10A USB3320, U10B USB3320, U10C USB3320, U10D USB3320, U11 MIC2025-1YMM, U12A USB3320, U12B USB3320, U12C USB3320, U12D USB3320, U20G xc7z020clg484, Y1 24.000MHZ, Y2 24.000MHZ

Commit message: Update audio schematic
Parts:
- renumbered U10A to U10A1, U10B to U10B1, U10C to U10C1, U10D to U10D1, U12A to U12A1, U12B to U12B1, U12C to U12C1, U12D to U12D1, U20G to U20G1
Changed lines of the file:
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@@
 		(on_board yes)
 		(dnp no)
-		(property "Reference" "U10A"
+		(property "Reference" "U10A1"
 			(at 123.19 26.67 0)
 			(effects
@@
 			(project "DFTBoard"
 				(path "/49eba173-d38c-4d05-b21c-b4a14c4948c2/00000000-0000-0000-0000-00005852a88e"
-					(reference "U10A")
+					(reference "U10A1")
 					(unit 1)
 				)
@@
 		(on_board yes)
 		(dnp no)
-		(property "Reference" "U10B"
+		(property "Reference" "U10B1"
 			(at 124.3076 103.8098 0)
 			(effects
@@
 			(project "DFTBoard"
 				(path "/49eba173-d38c-4d05-b21c-b4a14c4948c2/00000000-0000-0000-0000-00005852a88e"
-					(reference "U10B")
+					(reference "U10B1")
 					(unit 2)
 				)
@@
 		(on_board yes)
 		(dnp no)
-		(property "Reference" "U10C"
+		(property "Reference" "U10C1"
 			(at 147.4724 49.8602 0)
 			(effects
@@
 			(project "DFTBoard"
 				(path "/49eba173-d38c-4d05-b21c-b4a14c4948c2/00000000-0000-0000-0000-00005852a88e"
-					(reference "U10C")
+					(reference "U10C1")
 					(unit 3)
 				)
@@
 		(on_board yes)
 		(dnp no)
-		(property "Reference" "U10D"
+		(property "Reference" "U10D1"
 			(at 142.3924 25.7302 0)
 			(effects
@@
 			(project "DFTBoard"
 				(path "/49eba173-d38c-4d05-b21c-b4a14c4948c2/00000000-0000-0000-0000-00005852a88e"
-					(reference "U10D")
+					(reference "U10D1")
 					(unit 4)
 				)
@@
 		(on_board yes)
 		(dnp no)
-		(property "Reference" "U12A"
+		(property "Reference" "U12A1"
 			(at 218.44 29.21 0)
 			(effects
@@
 			(project "DFTBoard"
 				(path "/49eba173-d38c-4d05-b21c-b4a14c4948c2/00000000-0000-0000-0000-00005852a88e"
-					(reference "U12A")
+					(reference "U12A1")
 					(unit 1)
 				)
@@
 		(on_board yes)
 		(dnp no)
-		(property "Reference" "U12B"
+		(property "Reference" "U12B1"
 			(at 219.5576 106.3498 0)
 			(effects
@@
 			(project "DFTBoard"
 				(path "/49eba173-d38c-4d05-b21c-b4a14c4948c2/00000000-0000-0000-0000-00005852a88e"
-					(reference "U12B")
+					(reference "U12B1")
 					(unit 2)
 				)
@@
 		(on_board yes)
 		(dnp no)
-		(property "Reference" "U12C"
+		(property "Reference" "U12C1"
 			(at 242.7224 52.4002 0)
 			(effects
@@
 			(project "DFTBoard"
 				(path "/49eba173-d38c-4d05-b21c-b4a14c4948c2/00000000-0000-0000-0000-00005852a88e"
-					(reference "U12C")
+					(reference "U12C1")
 					(unit 3)
 				)
@@
 		(on_board yes)
 		(dnp no)
-		(property "Reference" "U12D"
+		(property "Reference" "U12D1"
 			(at 237.6424 28.2702 0)
 			(effects
@@
 			(project "DFTBoard"
 				(path "/49eba173-d38c-4d05-b21c-b4a14c4948c2/00000000-0000-0000-0000-00005852a88e"
-					(reference "U12D")
+					(reference "U12D1")
 					(unit 4)
 				)
@@
 		(on_board yes)
 		(dnp no)
-		(property "Reference" "U20G"
+		(property "Reference" "U20G1"
 			(at 75.7174 133.2738 0)
 			(effects
@@
 			(project "DFTBoard"
 				(path "/49eba173-d38c-4d05-b21c-b4a14c4948c2/00000000-0000-0000-0000-00005852a88e"
-					(reference "U20G")
+					(reference "U20G1")
 					(unit 7)
 				)
