File: zynqPCB/power.kicad_sch (KiCad schematic)
At the start: 60 parts, among them CON1 AVR-JTAG-10, U1 LM3880, U2 LM3880, U20A xc7z020clg484, U20I xc7z020clg484, U3 SC189 - 1.0V, U4 SC189 - 3.3V, U5 TLV62080DSGx, U7 SC189 - 1.8V

Commit message: Update audio schematic
Parts:
- renumbered U20A to U20A1, U20I to U20I1
Changed lines of the file:
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@@
 		(on_board yes)
 		(dnp no)
-		(property "Reference" "U20A"
+		(property "Reference" "U20A1"
 			(at 273.8374 77.3938 0)
 			(effects
@@
 			(project "DFTBoard"
 				(path "/49eba173-d38c-4d05-b21c-b4a14c4948c2/00000000-0000-0000-0000-000058508414"
-					(reference "U20A")
+					(reference "U20A1")
 					(unit 1)
 				)
@@
 		(on_board yes)
 		(dnp no)
-		(property "Reference" "U20I"
+		(property "Reference" "U20I1"
 			(at 278.9174 156.2862 0)
 			(effects
@@
 			(project "DFTBoard"
 				(path "/49eba173-d38c-4d05-b21c-b4a14c4948c2/00000000-0000-0000-0000-000058508414"
-					(reference "U20I")
+					(reference "U20I1")
 					(unit 9)
 				)
